Commit message: prismatic joint

File: urdf/urdfbot_simple.urdf (robot description, URDF)
Before this commit: robot urdfbot, 2 links, 1 joints
Joints:
- joint base_link_to_head_link_joint: axis (none) -> 0 0 1; limit (none) -> lower=-0.1 upper=0.1 effort=100 velocity=0.1; type fixed -> prismatic

Commit message: meshes in visual elements of links

File: urdf/urdfbot_simple.urdf (robot description, URDF)
Before this commit: robot urdfbot, 2 links, 1 joints
Links:
- link base_link: geometry visual mesh filename=package://urdfbot_description/meshes/urdfbot_body.dae scale=0.1 0.1 0.1
- link head_link: geometry visual mesh filename=package://urdfbot_description/meshes/urdfbot_head.dae scale=0.1 0.1 0.1
Joints:
- joint base_link_to_head_link_joint: limit lower=-0.1 upper=0.1 effort=100 velocity=0.1 -> lower=-1.57 upper=1.57 effort=100 velocity=1.0; origin xyz=0 0 0.11 rpy=0 0 0 -> xyz=0 0 0.07 rpy=0 0 0; type prismatic -> revolute

Commit message: robot with arm

File: urdf/urdfbot_simple.urdf (robot description, URDF)
Before this commit: robot urdfbot, 2 links, 1 joints
Links:
- added link claw_a_r_link; visual mesh filename=package://urdfbot_description/meshes/urdfbot_claw.dae scale=0.1 0.1 0.1
- added link claw_b_r_link; visual mesh filename=package://urdfbot_description/meshes/urdfbot_claw.dae scale=0.1 0.1 0.1
- added link lower_arm_r_link; visual mesh filename=package://urdfbot_description/meshes/urdfbot_limb.dae scale=0.1 0.1 0.1
- added link upper_arm_r_link; visual mesh filename=package://urdfbot_description/meshes/urdfbot_limb.dae scale=0.1 0.1 0.1
Joints:
- added joint base_link_to_upper_arm_r_link_joint: type revolute, parent base_link, child upper_arm_r_link, origin xyz=0 -0.03272 0.0279895 rpy=-1.57 0 0, axis 0 0 1, limit lower=-1.0 upper=1.0 effort=100 velocity=1.0
- added joint upper_arm_r_link_to_claw_a_r_link_joint: type revolute, parent lower_arm_r_link, child claw_a_r_link, origin xyz=0 0 -0.065 rpy=-1.57 0 -1.57, axis 0 0 1, limit lower=-0.7 upper=0.7 effort=100 velocity=1.0
- added joint upper_arm_r_link_to_claw_b_r_link_joint: type revolute, parent lower_arm_r_link, child claw_b_r_link, origin xyz=0 0 -0.065 rpy=-1.57 0 1.57, axis 0 0 1, limit lower=-0.7 upper=0.7 effort=100 velocity=1.0
- added joint upper_arm_r_link_to_lower_arm_r_link_joint: type revolute, parent upper_arm_r_link, child lower_arm_r_link, origin xyz=0 0 -0.0568 rpy=0 0 0, axis 1 0 0, limit lower=-1.0 upper=1.0 effort=100 velocity=1.0

Commit message: mimic element for robot claw fingers

File: urdf/urdfbot_simple.urdf (robot description, URDF)
Before this commit: robot urdfbot, 6 links, 5 joints
Joints:
- joint upper_arm_r_link_to_claw_b_r_link_joint: mimic (none) -> joint=upper_arm_r_link_to_claw_a_r_link_joint multiplier=1.0 offset=0.0
